File: Eagel/KranPowerV2_1.brd (EAGLE design)
At the start: 100 x 100 mm, 71 parts, among them IC1 INA138, IC2 INA138, IC3 INA138, IC4 INA138, IC5 INA138, IC6 INA138, IC7 4017D, IC8 MCP3008, IC9 7805, Q1 BSS123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

Commit message: small update
Parts:
- added C22: (no value), rcl:C0603
- added C23: (no value), rcl:SMC_B
- added LOGO1: OSHW_LOGO_FILLX0350-NT, ohw-logo:OSHW_FILLX350_NOTEXT
- added U$13: KRAN_LOGO, MWlogo:KRAN_LOGO
- added U$14: (no value), MWlogo:KRAN_LOGO_STOP
- C10, C11, C7, C8, C9: value (none) -> 1u
- U1: value DS26LS31CM -> DS26LS31
- moved C6 1.91 mm to (24.1, 83.8)
- moved R2 1.91 mm to (24.1, 85.7)
Connections:
- net +5V: now also C22.1, C23.+
- net GND: now also C22.2, C23.-
Routing:
- net GND: track 54.1 -> 56.6 mm, vias 11 -> 13
- net +5V: track 242.0 -> 244.3 mm
- net N$9: track 19.8 -> 21.1 mm
- net N$7: track 19.5 -> 20.8 mm
- net N$11: track 18.7 -> 19.6 mm
- net CS_TFT: track 65.4 -> 64.8 mm
- net MOSI: track 126.6 -> 126.0 mm
Other:
- board text added: "1"
- board text added: "100n 50k"
- board text added: "10k"
- board text added: "1k"
- board text added: "1u"
- board text added: "2"
- board text added: "25A"
- board text added: "3"
- board text added: "4"
- board text added: "5"
- board text added: "5,6V"
- board text added: "6"
- board text added: "74HC4017"
- board text added: "Aus"
- board text added: "B"
- board text added: "BSS138"
- board text added: "CTS"
- board text added: "DRT"
- board text added: "DS26LS31"
- board text added: "GND"
- board text added: "Kran Power V2.1"
- board text added: "MCP3008"
- board text added: "Not"
- board text added: "O"
- board text added: "R"
- board text added: "RXI"
- board text added: "TXD"
- board text added: "VCC"
- board text removed: "Kran Steuerung V2.1"
