File: Eagel/KranPowerV2_1.brd (EAGLE design)
At the start: 100 x 100 mm, 76 parts, among them IC1 INA138, IC2 INA138, IC3 INA138, IC4 INA138, IC5 INA138, IC6 INA138, IC7 4017D, IC8 MCP3008, IC9 7805, Q1 BSS123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

Commit message: small update
Routing:
- net GND: track 56.6 -> 149.4 mm
Changed lines of the file:
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@@
 <via x="97.79" y="91.44" extent="1-16" drill="0.9" diameter="1.6764" shape="octagon"/>
 <wire x1="97.79" y1="93.98" x2="97.79" y2="91.44" width="0.4064" layer="16"/>
+<wire x1="26.035" y1="40.005" x2="26.035" y2="44.7675" width="1.778" layer="16"/>
+<wire x1="26.035" y1="44.7675" x2="26.035" y2="50.8" width="1.778" layer="16"/>
+<wire x1="26.035" y1="50.8" x2="24.765" y2="50.8" width="1.778" layer="16"/>
+<wire x1="24.765" y1="50.8" x2="22.86" y2="48.895" width="1.778" layer="16"/>
+<wire x1="48.895" y1="50.8" x2="48.895" y2="44.45" width="1.778" layer="16"/>
+<wire x1="48.895" y1="44.45" x2="48.895" y2="40.64" width="1.778" layer="16"/>
+<wire x1="67.945" y1="5.08" x2="71.755" y2="5.08" width="1.778" layer="16"/>
+<wire x1="71.755" y1="5.08" x2="71.755" y2="1.905" width="1.778" layer="16"/>
+<wire x1="45.085" y1="5.08" x2="48.895" y2="5.08" width="1.778" layer="16"/>
+<wire x1="48.895" y1="5.08" x2="48.895" y2="1.905" width="1.778" layer="16"/>
+<wire x1="22.225" y1="5.08" x2="26.035" y2="5.08" width="1.778" layer="16"/>
+<wire x1="26.035" y1="5.08" x2="26.035" y2="2.54" width="1.778" layer="16"/>
+<wire x1="71.755" y1="50.8" x2="71.755" y2="44.45" width="1.778" layer="16"/>
+<wire x1="71.755" y1="44.45" x2="68.58" y2="41.275" width="1.778" layer="16"/>
+<wire x1="71.12" y1="50.8" x2="69.215" y2="50.8" width="1.778" layer="16"/>
+<wire x1="71.755" y1="5.08" x2="75.565" y2="5.08" width="1.778" layer="16"/>
+<wire x1="72.39" y1="90.805" x2="73.66" y2="90.805" width="1.778" layer="16"/>
+<wire x1="73.66" y1="90.805" x2="74.93" y2="92.075" width="1.778" layer="16"/>
+<wire x1="71.755" y1="90.805" x2="71.755" y2="91.44" width="1.778" layer="16"/>
+<wire x1="71.755" y1="91.44" x2="70.485" y2="92.71" width="1.778" layer="16"/>
+<wire x1="48.895" y1="89.535" x2="48.895" y2="88.265" width="1.778" layer="16"/>
+<wire x1="48.895" y1="88.265" x2="49.53" y2="87.63" width="1.778" layer="16"/>
+<wire x1="48.895" y1="90.805" x2="48.895" y2="93.98" width="1.778" layer="16"/>
+<wire x1="26.035" y1="90.805" x2="26.035" y2="92.71" width="1.778" layer="16"/>
+<wire x1="26.035" y1="92.71" x2="27.305" y2="93.98" width="1.778" layer="16"/>
+<wire x1="26.035" y1="90.805" x2="27.94" y2="90.805" width="1.778" layer="16"/>
+<wire x1="26.035" y1="90.805" x2="26.035" y2="88.265" width="1.778" layer="16"/>
+<wire x1="26.035" y1="88.265" x2="26.67" y2="87.63" width="1.778" layer="16"/>
+<wire x1="48.895" y1="50.8" x2="50.8" y2="50.8" width="1.778" layer="16"/>
+<wire x1="48.895" y1="44.45" x2="51.1175" y2="44.45" width="1.778" layer="16"/>
+<wire x1="26.035" y1="44.7675" x2="23.495" y2="44.7675" width="1.778" layer="16"/>
+<wire x1="48.895" y1="5.08" x2="51.1175" y2="5.08" width="1.778" layer="16"/>
+<wire x1="26.035" y1="5.08" x2="28.2575" y2="5.08" width="1.778" layer="16"/>
 </signal>
 <signal name="P_OUT1">
