File: Eagel/KranPowerV2_1.sch (EAGLE design)
At the start: 69 parts, among them IC1 INA138, IC2 INA138, IC3 INA138, IC4 INA138, IC5 INA138, IC6 INA138, IC7 4017D, IC8 MCP3008, IC9 7805, Q1 BSS123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

Commit message: small update
Parts:
- added C22: (no value), rcl:C-EUC0603
- added C23: (no value), rcl:CPOL-EUSMCB
- added LOGO1: OSHW_LOGO_FILLX0350-NT, ohw-logo:OSHW_LOGO_FILLX0350-NT
- added U$13: KRAN_LOGO, MWlogo:KRAN_LOGO
- C10, C11, C7, C8, C9: value (none) -> 1u
- U1: value DS26LS31CM -> DS26LS31
Connections:
- net +5V: now also C22.1, C23.+
- net GND: now also C22.2, C23.-
Other:
- moved on the sheet: C21, C5, IC7P
Changed lines of the file:
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@@
 <part name="U$3" library="MWlogo" deviceset="KRAN_LOGO" device=""/>
 <part name="C6" library="rcl" deviceset="C-EU" device="C0603" value="1u"/>
-<part name="C7" library="rcl" deviceset="C-EU" device="C0603"/>
-<part name="C8" library="rcl" deviceset="C-EU" device="C0603"/>
-<part name="C9" library="rcl" deviceset="C-EU" device="C0603"/>
-<part name="C10" library="rcl" deviceset="C-EU" device="C0603"/>
-<part name="C11" library="rcl" deviceset="C-EU" device="C0603"/>
+<part name="C7" library="rcl" deviceset="C-EU" device="C0603" value="1u"/>
+<part name="C8" library="rcl" deviceset="C-EU" device="C0603" value="1u"/>
+<part name="C9" library="rcl" deviceset="C-EU" device="C0603" value="1u"/>
+<part name="C10" library="rcl" deviceset="C-EU" device="C0603" value="1u"/>
+<part name="C11" library="rcl" deviceset="C-EU" device="C0603" value="1u"/>
 <part name="P+5" library="supply1" deviceset="+12V" device=""/>
 <part name="P+6" library="supply1" deviceset="+12V" device=""/>
@@
 <part name="C17" library="rcl" deviceset="C-EU" device="C0603" value="100n"/>
 <part name="GND32" library="supply1" deviceset="GND" device=""/>
-<part name="U1" library="Matthias" deviceset="DS26LS31CM" device=""/>
+<part name="U1" library="Matthias" deviceset="DS26LS31CM" device="" value="DS26LS31"/>
 <part name="GND33" library="supply1" deviceset="GND" device=""/>
 <part name="P+9" library="supply1" deviceset="+5V" device=""/>
@@
 <part name="P+11" library="supply1" deviceset="+5V" device=""/>
 <part name="D4" library="diode" deviceset="BY251" device=""/>
+<part name="C22" library="rcl" deviceset="C-EU" device="C0603"/>
+<part name="C23" library="rcl" deviceset="CPOL-EU" device="SMCB"/>
+<part name="U$13" library="MWlogo" deviceset="KRAN_LOGO" device=""/>
+<part name="LOGO1" library="ohw-logo" deviceset="OSHW_LOGO_FILL" device="X0350-NT"/>
 </parts>
 <sheets>
@@
 <instance part="GND3" gate="1" x="33.02" y="205.74"/>
 <instance part="U$1" gate="G$1" x="261.62" y="210.82" rot="MR0"/>
-<instance part="IC7" gate="P" x="157.48" y="38.1"/>
+<instance part="IC7" gate="P" x="172.72" y="38.1"/>
 <instance part="GND19" gate="1" x="314.96" y="162.56"/>
 <instance part="GND20" gate="1" x="119.38" y="27.94"/>
@@
 <instance part="C19" gate="G$1" x="66.04" y="71.12"/>
 <instance part="C20" gate="G$1" x="35.56" y="71.12"/>
-<instance part="C21" gate="G$1" x="142.24" y="40.64"/>
-<instance part="C5" gate="G$1" x="149.86" y="40.64"/>
+<instance part="C21" gate="G$1" x="157.48" y="40.64"/>
+<instance part="C5" gate="G$1" x="165.1" y="40.64"/>
 <instance part="U$5" gate="G$1" x="50.8" y="33.02"/>
 <instance part="U$5" gate="G$2" x="27.94" y="210.82"/>
@@
 <instance part="P+11" gate="1" x="312.42" y="109.22"/>
 <instance part="D4" gate="1" x="43.18" y="40.64"/>
+<instance part="C22" gate="G$1" x="142.24" y="40.64"/>
+<instance part="C23" gate="G$1" x="149.86" y="40.64"/>
+<instance part="U$13" gate="G$1" x="45.72" y="10.16"/>
+<instance part="LOGO1" gate="G$1" x="68.58" y="17.78"/>
 </instances>
 <busses>
@@
 <pinref part="IC7" gate="P" pin="VSS"/>
 <pinref part="GND20" gate="1" pin="GND"/>
+<wire x1="172.72" y1="30.48" x2="165.1" y2="30.48" width="0.1524" layer="91"/>
+<pinref part="C1" gate="G$1" pin="2"/>
+<wire x1="165.1" y1="30.48" x2="157.48" y2="30.48" width="0.1524" layer="91"/>
 <wire x1="157.48" y1="30.48" x2="149.86" y2="30.48" width="0.1524" layer="91"/>
-<pinref part="C1" gate="G$1" pin="2"/>
 <wire x1="149.86" y1="30.48" x2="142.24" y2="30.48" width="0.1524" layer="91"/>
 <wire x1="142.24" y1="30.48" x2="134.62" y2="30.48" width="0.1524" layer="91"/>
@@
 <junction x="134.62" y="30.48"/>
 <pinref part="C21" gate="G$1" pin="-"/>
+<wire x1="157.48" y1="35.56" x2="157.48" y2="30.48" width="0.1524" layer="91"/>
+<junction x="157.48" y="30.48"/>
+<pinref part="C5" gate="G$1" pin="-"/>
+<wire x1="165.1" y1="35.56" x2="165.1" y2="30.48" width="0.1524" layer="91"/>
+<junction x="165.1" y="30.48"/>
+<pinref part="C22" gate="G$1" pin="2"/>
 <wire x1="142.24" y1="35.56" x2="142.24" y2="30.48" width="0.1524" layer="91"/>
 <junction x="142.24" y="30.48"/>
-<pinref part="C5" gate="G$1" pin="-"/>
+<pinref part="C23" gate="G$1" pin="-"/>
 <wire x1="149.86" y1="35.56" x2="149.86" y2="30.48" width="0.1524" layer="91"/>
 <junction x="149.86" y="30.48"/>
@@
 <pinref part="IC7" gate="P" pin="VDD"/>
 <pinref part="P+2" gate="1" pin="+5V"/>
+<wire x1="172.72" y1="45.72" x2="165.1" y2="45.72" width="0.1524" layer="91"/>
+<pinref part="C1" gate="G$1" pin="1"/>
+<wire x1="165.1" y1="45.72" x2="157.48" y2="45.72" width="0.1524" layer="91"/>
 <wire x1="157.48" y1="45.72" x2="149.86" y2="45.72" width="0.1524" layer="91"/>
-<pinref part="C1" gate="G$1" pin="1"/>
 <wire x1="149.86" y1="45.72" x2="142.24" y2="45.72" width="0.1524" layer="91"/>
 <wire x1="142.24" y1="45.72" x2="134.62" y2="45.72" width="0.1524" layer="91"/>
@@
 <junction x="134.62" y="45.72"/>
 <pinref part="C21" gate="G$1" pin="+"/>
-<wire x1="142.24" y1="43.18" x2="142.24" y2="45.72" width="0.1524" layer="91"/>
+<wire x1="157.48" y1="43.18" x2="157.48" y2="45.72" width="0.1524" layer="91"/>
+<junction x="157.48" y="45.72"/>
+<pinref part="C5" gate="G$1" pin="+"/>
+<wire x1="165.1" y1="43.18" x2="165.1" y2="45.72" width="0.1524" layer="91"/>
+<junction x="165.1" y="45.72"/>
+<pinref part="C22" gate="G$1" pin="1"/>
+<wire x1="142.24" y1="45.72" x2="142.24" y2="43.18" width="0.1524" layer="91"/>
 <junction x="142.24" y="45.72"/>
-<pinref part="C5" gate="G$1" pin="+"/>
+<pinref part="C23" gate="G$1" pin="+"/>
 <wire x1="149.86" y1="43.18" x2="149.86" y2="45.72" width="0.1524" layer="91"/>
 <junction x="149.86" y="45.72"/>
